File: Schematic/Clave.kicad_sch (KiCad schematic)
At the start: 48 parts, among them Q1101 BC847, Q1102 BC856, Q1103 BC847, Q1104 BC847, Q1105 MPF4393, U1101 TL072, U1102 TL071

Commit message: rev. 2 schematic and board
Parts:
- Q1105: footprint Package_TO_SOT_THT:TO-92L_HandSolder -> Package_TO_SOT_THT:TO-92L
