File: Schematic/MCU.kicad_sch (KiCad schematic)
At the start: 25 parts, among them J401 Micro_SD_Card_Det2, SW401 BOOT, SW402 RST, U401 ESP32-S3-WROOM-1, U402 TL072, U403 PCM5100A, U404 MSP4331-20Pin, U405 MSP4331-20Pin

Commit message: rev. 2 schematic and board
Parts:
- added R404, R405, R406: 47k, PCM_Resistor_SMD_AKL:R_0805_2012Metric, symbol Device:R_US
Connections:
- net +3.3V: now also R404.1, R405.1, R406.1
- net POT1_CS: now also U401.35 (MTMS/GPIO42), R405.2; no longer U401.34 (MTDI/GPIO41/CLK_OUT1)
- net POT2_CS: now also U401.34 (MTDI/GPIO41/CLK_OUT1), R406.2; no longer U401.35 (MTMS/GPIO42)
- net SD_CS: now also R404.2
- net IO19 renamed USB-
- net IO20 renamed USB+
Other:
- moved on the sheet: J401

Commit message: pins
Parts:
- U404, U405: value MSP4331-20Pin -> MCP4331-20Pin
