File: Schematic/Controls.kicad_sch (KiCad schematic)
At the start: 66 parts, among them SW201 SW_SPST, SW202 SW_SPST, SW203 SW_SPST, SW204 SW_SPST, SW205 SW_SPST, SW206 SW_SPST, SW207 SW_SPST, SW208 SW_SPST, SW209 SW_SPST, SW210 SW_SPST, SW211 SW_SPST, SW212 SW_SPST, SW213 SW_SPST, SW214 SW_SPST, SW215 SW_SPST, SW216 SW_SPST, SW217 SW_SPST, SW218 SW_SPST, SW219 LOAD, SW220 SAVE, SW221 TrackSel, SW222 Digital1, SW223 Digital2, SW224 Digital3, SW225 PLAYTOGGLE, SW226 ALT, U201 MCP23S17_SO, U202 MCP23S17_SO, U205 MCP23S17_SO

Commit message: rev. 2 schematic and board
Parts:
- added R201, R202: 47k, PCM_Resistor_SMD_AKL:R_0805_2012Metric, symbol Device:R_US
Connections:
- net +3.3V: now also R201.1, R202.1
- net ALT: now also U205.24 (GPA3); no longer U205.22 (GPA1)
- net D_CS: now also R201.2
- net EXP_CS: now also R202.2
- net LOAD: now also U205.21 (GPA0); no longer U205.23 (GPA2)
- net PLAYTOGGLE: now also U205.23 (GPA2); no longer U205.21 (GPA0)
- net SAVE: now also U205.22 (GPA1); no longer U205.24 (GPA3)
Other:
- moved on the sheet: U203

Commit message: naming stuff, bit packing stuff
Parts:
- U201, U202, U205: value MCP23S17_SO -> Adafruit_MCP23X17_SO; symbol Interface_Expansion:MCP23S17_SO -> Interface_Expansion:Adafruit_MCP23X17_SO
Changed lines of the file:
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@@
     )
   )
-  (symbol (lib_id "Interface_Expansion:MCP23S17_SO") (at 430.53 144.78 0) (unit 1)
+  (symbol (lib_id "Interface_Expansion:Adafruit_MCP23X17_SO") (at 430.53 144.78 0) (unit 1)
     (in_bom yes) (on_board yes) (dnp no) (fields_autoplaced)
     (property "Reference" "U202" (at 432.7241 117.475 0)
       (effects (font (size 1.27 1.27)) (justify left))
     )
-    (property "Value" "MCP23S17_SO" (at 432.7241 120.015 0)
+    (property "Value" "Adafruit_MCP23X17_SO" (at 432.7241 120.015 0)
       (effects (font (size 1.27 1.27)) (justify left))
     )
@@
     )
   )
-  (symbol (lib_id "Interface_Expansion:MCP23S17_SO") (at 430.53 72.39 0) (unit 1)
+  (symbol (lib_id "Interface_Expansion:Adafruit_MCP23X17_SO") (at 430.53 72.39 0) (unit 1)
     (in_bom yes) (on_board yes) (dnp no) (fields_autoplaced)
     (property "Reference" "U201" (at 432.7241 45.085 0)
       (effects (font (size 1.27 1.27)) (justify left))
     )
-    (property "Value" "MCP23S17_SO" (at 432.7241 47.625 0)
+    (property "Value" "Adafruit_MCP23X17_SO" (at 432.7241 47.625 0)
       (effects (font (size 1.27 1.27)) (justify left))
     )
@@
     )
   )
-  (symbol (lib_id "Interface_Expansion:MCP23S17_SO") (at 429.895 217.805 0) (unit 1)
+  (symbol (lib_id "Interface_Expansion:Adafruit_MCP23X17_SO") (at 429.895 217.805 0) (unit 1)
     (in_bom yes) (on_board yes) (dnp no) (fields_autoplaced)
     (property "Reference" "U205" (at 432.0891 190.5 0)
       (effects (font (size 1.27 1.27)) (justify left))
     )
-    (property "Value" "MCP23S17_SO" (at 432.0891 193.04 0)
-      (effects (font (size 1.27 1.27)) (justify left))
-    )
+    (property "Value" "Adafruit_MCP23X17_SO" (at 432.0891 193.04 0)
+      (effects (font (size 1.27 1.27)) (justify left))
+    )
