File: Schematic/PowerSupply.kicad_sch (KiCad schematic)
At the start: 46 parts, among them J302 USB_B_Micro, J502 BATTERY, J503 POWER, Q501 SQ2315, Q502 SQ2315, U501 MAX1898, U502 TPS61200DRC, U503 CS5173, U504 LTC1044

Commit message: rev. 2 schematic and board
Parts:
- FB501: value FerriteBead -> 600R
- Q501, Q502: value SQ2315 -> Q_PMOS_GSD; footprint PCM_Package_TO_SOT_SMD_AKL:SOT-23 -> PCM_4ms_Package_SOT:SOT-23; symbol Device:Q_PMOS_GDS -> Device:Q_PMOS_GSD
Connections:
- net +3.3V: now also U502.8 (PS); no longer D504.2 (A)
- net BATT+: now also Q502.2 (S); no longer Q502.3 (S)
- net GND: no longer U502.8 (PS)
- net VCC: now also Q502.3 (D); no longer Q502.2 (D)
- net at L502.1, U503.8 (Vsw): now also D504.2 (A)
- net at U501.10 (CS): now also Q501.3 (D); no longer Q501.2 (D)
- net at D503.2 (A): now also Q501.2 (S); no longer Q501.3 (S)
- net IO19 renamed USB-
- net IO20 renamed USB+
Other:
- note removed: "NOTE: Change this footprint to GSD layout because GDS mosfets apparently don't exist"
- moved on the sheet: C507, D504, L502, R503, R504

Commit message: battery monitoring stuff
Parts:
- R512: value 15k -> 33k
Other:
- note added: "According to the datasheet, this can work with inputs as low as 300mV, so we'll set our 0% battery in software at ~400mV to be safe"
- note added: "The MAX1898 will charge the battery to 4.1v, which means the max voltage at BATT_REF is about 3.083v"
Changed lines of the file:
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@@
     (fill (type none))
   )
-  (rectangle (start 18.415 21.59) (end 141.605 93.345)
+  (rectangle (start 18.415 21.59) (end 164.973 93.345)
     (stroke (width 0) (type solid))
     (fill (type none))
   )
+  (text "According to the datasheet,\nthis can work with inputs \nas low as 300mV, so we'll \nset our 0% battery in\nsoftware at ~400mV to be safe"
+    (at 74.295 115.062 0)
+    (effects (font (size 1.27 1.27)) (justify left bottom))
+  )
   (text "+12v to -12v charge \npump inverter" (at 204.216 109.982 0)
     (effects (font (size 2.032 2.032)) (justify left bottom))
@@
   (text "Battery Charger" (at 18.415 20.32 0)
     (effects (font (size 3.81 3.81) (thickness 0.762) bold) (justify left bottom))
+  )
+  (text "The MAX1898 will charge the\nbattery to 4.1v, which means \nthe max voltage at BATT_REF \nis about 3.083v"
+    (at 133.477 75.057 0)
+    (effects (font (size 1.27 1.27)) (justify left bottom))
   )
   (text "This sets the charging \ncurrent at ~298 mA" (at 66.675 66.04 0)
@@
       (effects (font (size 1.27 1.27)) (justify left))
     )
-    (property "Value" "15k" (at 115.57 73.025 0)
-      (effects (font (size 1.27 1.27)) (justify left))
-    )
+    (property "Value" "33k" (at 115.57 73.025 0)
+      (effects (font (size 1.27 1.27)) (justify left))
+    )
